File: keyboard unit ruler.kicad_pcb (KiCad board)
At the start: 2 copper layers, 252.4 x 19.1 mm, 23 parts

Commit message: Added URl
Other:
- board text added: "https://github.com/Technofrikus/keyboard-unit-pcb-ruler"
